File: STM32/STM32.kicad_sch (KiCad schematic)
At the start: 28 parts, among them J1 USB_B_Micro, J2 Conn_01x04_Pin, J3 Conn_01x04_Pin, J4 Conn_01x04_Pin, SW1 SW_SPDT, U1 AMS1117-3.3, U2 STM32F103C8T6, Y1 16MHz

Commit message: Add files via upload
Other:
- company: Phil's Lab -> ROOPA GHATKE
Changed lines of the file:
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@@
 		(date "2025-07-21")
 		(rev "0.1")
-		(company "Phil's Lab")
+		(company "ROOPA GHATKE")
 	)
 	(text "STM32 MCU PCB\n"
